Commit message: Apparently the collision name warning is real

File: wamv_description/urdf/battery.xacro (robot description, xacro)
@@ -9,5 +9,5 @@
         </geometry>
       </visual>
-      <collision name="${prefix}_battery_collision">
+      <collision>
         <origin xyz="0 0 .15" rpy="0 0 0"/>
         <geometry>

File: wamv_description/urdf/cpu_cases.xacro (robot description, xacro)
@@ -9,5 +9,5 @@
       </geometry>
     </visual>
-    <collision name="cpu_case_1_collision">
+    <collision>
       <origin xyz="0.185 0 0" rpy="0 0 0"/>
       <geometry>
@@ -15,5 +15,5 @@
       </geometry>
     </collision>
-    <collision name="cpu_case_2_collision">
+    <collision>
       <origin xyz="-0.3 0 -0.092" rpy="0 0 0"/>
       <geometry>

File: wamv_description/urdf/thrusters/engine.xacro (robot description, xacro)
@@ -9,5 +9,5 @@
         </geometry>
       </visual>
-      <collision name="${prefix}_engine_vertical_axis_collision">
+      <collision>
         <origin xyz="-0.16 0 -0.24" rpy="0 0 0" />
         <geometry>
@@ -15,5 +15,5 @@
         </geometry>
       </collision>
-      <collision name="${prefix}_engine_rear_end_collision">
+      <collision>
         <origin xyz="-0.34 0 0.12" rpy="0 0 0" />
         <geometry>
@@ -32,5 +32,5 @@
         </geometry>
       </visual>
-      <collision name="${prefix}_propeller_collision">
+      <collision>
         <origin xyz="-0.08 0 0" rpy="0 1.57 0" />
         <geometry>

File: wamv_description/urdf/wamv_base.urdf.xacro (robot description, xacro)
@@ -4,5 +4,5 @@
   <xacro:macro name="main_collisions" params="prefix reflect:=1">
     <!-- Main float -->
-    <collision name="${prefix}_float">
+    <collision>
       <origin xyz="-0.4 ${1.03*reflect} 0.2" rpy="${0*reflect} 1.57 0" />
       <geometry>
@@ -10,5 +10,5 @@
       </geometry>
     </collision>
-    <collision name="${prefix}_mid_float">
+    <collision>
       <origin xyz="1.85 ${1.03*reflect} 0.3" rpy="${0*reflect} 1.38 0" />
       <geometry>
@@ -16,5 +16,5 @@
       </geometry>
     </collision>
-    <collision name="${prefix}_front_float">
+    <collision>
       <origin xyz="2.3 ${1.03*reflect} 0.4" rpy="${0*reflect} 1.3 0" />
       <geometry>
@@ -23,5 +23,5 @@
     </collision>
     <!-- Front beam -->
-    <collision name="front_${prefix}_beam_lower">
+    <collision>
       <origin xyz="0.9 ${0.85*reflect} 1" rpy="${0.78*reflect} 0 0" />
       <geometry>
@@ -29,5 +29,5 @@
       </geometry>
     </collision>
-    <collision name="front_${prefix}_beam_upper">
+    <collision>
       <origin xyz="0.9 ${0.6*reflect} 1.18" rpy="${1.35*reflect} 0 0" />
       <geometry>
@@ -36,5 +36,5 @@
     </collision>
     <!-- Mid beam -->
-    <collision name="mid_${prefix}_beam_lower">
+    <collision>
       <origin xyz="-0.65 ${0.99*reflect} 0.7" rpy="${0.1*reflect} 0.25 0" />
       <geometry>
@@ -42,5 +42,5 @@
       </geometry>
     </collision>
-    <collision name="mid_${prefix}_beam_medium">
+    <collision>
       <origin xyz="-0.57 ${0.87*reflect} 1.05" rpy="${0.75*reflect} 0.25 0" />
       <geometry>
@@ -48,5 +48,5 @@
       </geometry>
     </collision>
-    <collision name="mid_${prefix}_beam_upper">
+    <collision>
       <origin xyz="-0.55 ${0.65*reflect} 1.17" rpy="${1.35*reflect} 0.25 0" />
       <geometry>
@@ -55,5 +55,5 @@
     </collision>
     <!-- Rear beam -->
-    <collision name="rear_${prefix}_beam_lower">
+    <collision>
       <origin xyz="-0.74 ${1.03*reflect} 0.7" rpy="${0*reflect} -0.15 0" />
       <geometry>
@@ -61,5 +61,5 @@
       </geometry>
     </collision>
-    <collision name="rear_${prefix}_beam_medium">
+    <collision>
       <origin xyz="-0.79 ${0.91*reflect} 1.05" rpy="${0.75*reflect} -0.15 0" />
       <geometry>
@@ -67,5 +67,5 @@
       </geometry>
     </collision>
-    <collision name="rear_${prefix}_beam_upper">
+    <collision>
       <origin xyz="-0.81 ${0.67*reflect} 1.18" rpy="${1.45*reflect} -0.15 0" />
       <geometry>
@@ -74,5 +74,5 @@
     </collision>
     <!-- Joint -->
-    <collision name="${prefix}_joint">
+    <collision>
       <origin xyz="0.58 ${1.03*reflect} 0.6" rpy="${0*reflect} -0.6 0" />
       <geometry>
@@ -99,5 +99,5 @@
     <xacro:main_collisions prefix="right" reflect="-1" />
      <!-- Top base -->
-    <collision name="top_base">
+    <collision>
       <origin xyz="0 -0 1.25" rpy="0 0 0" />
       <geometry>

File: wamv_gazebo/urdf/sensors/wamv_3d_lidar.xacro (robot description, xacro)
@@ -42,5 +42,5 @@
         </geometry>
       </visual>
-      <collision name="${name}_collision">
+      <collision>
         <geometry>
           <cylinder radius="0.055" length="0.075"/>
@@ -73,5 +73,5 @@
         </material>
       </visual>
-      <collision name="${name}_post_collision">
+      <collision>
         <geometry>
           <cylinder radius="${post_radius}" length="${post_length}"/>
@@ -97,5 +97,5 @@
         </geometry>
       </visual>
-      <collision name="${name}_post_arm_collision">
+      <collision>
         <origin xyz="0 0 0" rpy="${radians(-60)-pi/20} 0 ${-pi/2}"/>
         <geometry>

File: wamv_gazebo/urdf/sensors/wamv_camera.xacro (robot description, xacro)
@@ -15,5 +15,5 @@
         </geometry>
       </visual>
-      <collision name="${name}_lens_collision">
+      <collision>
         <origin xyz="0.018 0 0" rpy="0 ${pi/2} 0"/>
         <geometry>
@@ -21,5 +21,5 @@
         </geometry>
       </collision>
-      <collision name="${name}_box_collision">
+      <collision>
         <origin xyz="-0.0205 0 0" rpy="0 0 0"/>
         <geometry>
@@ -58,5 +58,5 @@
         </material>
       </visual>
-      <collision name="${name}_post_collision">
+      <collision>
         <geometry>
           <cylinder radius="${post_radius}" length="${post_length}"/>
@@ -82,5 +82,5 @@
         </geometry>
       </visual>
-      <collision name="${name}_post_arm_collision">
+      <collision>
         <origin xyz="0 0 0" rpy="${radians(-60)-pi/20} 0 ${-pi/2}"/>
         <geometry>

File: wamv_gazebo/urdf/sensors/wamv_gps.xacro (robot description, xacro)
@@ -8,5 +8,5 @@
         </geometry>
       </visual>
-      <collision name="${name}_collision_base">
+      <collision>
         <origin xyz="0 0 0.025" rpy="0 0 0" />
         <geometry>
@@ -14,5 +14,5 @@
         </geometry>
       </collision>
-      <collision name="${name}_collision_antenna">
+      <collision>
         <origin xyz="0 0 0.11" rpy="0 0 0" />
         <geometry>

File: wamv_gazebo/urdf/sensors/wamv_pinger.xacro (robot description, xacro)
@@ -9,5 +9,5 @@
         </geometry>
       </visual>
-      <collision name="${name}_collision">
+      <collision>
         <origin xyz="0 0 0" rpy="0 0 0" />
         <geometry>
