Commit message: added drone pad and cpu cases

File: wamv_description/urdf/wamv_base.urdf.xacro (robot description, xacro)
@@ -114,3 +114,31 @@
     </inertial>
   </link>
+  <gazebo reference="${namespace}/drone_pad">
+    <material>Gazebo/Gray</material>
+  </gazebo>
+  <link name="${namespace}/drone_pad">
+    <visual>
+      <origin xyz="-1.35 0 1.25" rpy="0 0 0" />
+      <geometry>
+        <box size="1 1 0.05" />
+      </geometry>
+    </visual>
+     <!-- Top base -->
+    <collision>
+      <origin xyz="-1.35 0 1.25" rpy="0 0 0" />
+      <geometry>
+        <box size="1 1 0.05" />
+      </geometry>
+    </collision>
+    <inertial>
+      <!-- From WAM-V spec sheet -->
+      <!--TODO: add mass and inertia of this link whenever it is added to NaviGator-->
+      <mass value="0.0"/>
+      <inertia ixx="120.0" ixy="0.0" ixz="0.0" iyy="393" iyz="0.0" izz="446.0"/>
+    </inertial>
+  </link>
+  <joint name="${namespace}/dummy_joint2" type = "fixed">
+    <parent link="${namespace}/dummy_link"/>
+    <child link="${namespace}/drone_pad"/>
+  </joint>
 </robot>

File: wamv_gazebo/urdf/wamv_gazebo.urdf.xacro (robot description, xacro)
@@ -93,6 +93,6 @@
     <xacro:yaml_components />
     <!-- Add CPU Cases -->
-    <!--<xacro:include filename="$(find wamv_description)/urdf/cpu_cases.xacro" />
-    <xacro:cpu_cases position="-0.15 0 1.53" orientation="0 0 0"/>-->
+    <xacro:include filename="$(find wamv_description)/urdf/cpu_cases.xacro" />
+    <xacro:cpu_cases position="-0.15 0 1.53" orientation="0 0 0"/>
   </xacro:if>
   <!-- Otherwise, add sensors based on enable variables -->
