Commit message: updated vrx code

File: vrx_gazebo/worlds/example_course.world.xacro (robot description, xacro)
@@ -1,33 +1,11 @@
 <?xml version="1.0" ?>
-<!-- World containing sandisland model and some course challenges -->
+<!-- World containing sydneyregatta model and some course challenges -->
 <sdf version="1.6" xmlns:xacro="http://ros.org/wiki/xacro">
   <world name="robotx_example_course">
-    <xacro:include filename="$(find vrx_gazebo)/worlds/sandisland.xacro" />
-    <xacro:sandisland />
+    <xacro:include filename="$(find vrx_gazebo)/worlds/sydneyregatta.xacro" />
+    <xacro:sydneyregatta />
     <!--Waves-->
     <xacro:include filename="$(find wave_gazebo)/world_models/ocean_waves/model.xacro"/>
-    <xacro:ocean_waves/>
-    <include>
-      <uri>model://robotx_navigation_challenge</uri>
-      <pose>58 68 2 0 0 0.4</pose>
-    </include>
-    <include>
-      <uri>model://robotx_light_buoy</uri>
-      <pose>110 28 0.25 0 0 0</pose>
-    </include>
-    <include>
-      <uri>model://robotx_2016_qualifying_pinger_transit</uri>
-      <pose>55 -50 0 0 0 -1.3</pose>
-    </include>
-    <!-- The 2016 dock with the three placards -->
-    <include>
-      <uri>model://dock_2016</uri>
-      <pose>75 22 0.0 0 0 -2.78</pose>
-    </include>
-    <!-- The 2018 dock with the two placards -->
-    <include>
-      <uri>model://dock_2018</uri>
-      <pose>-2 -18 0.0 0 0 0.2</pose>
-    </include>
+    <xacro:ocean_waves scale="2.5"/>
     <xacro:include filename="$(find vrx_gazebo)/worlds/xacros/usv_wind_plugin.xacro"/>
     <xacro:usv_wind_gazebo>
@@ -35,5 +13,5 @@
         <wind_obj>
           <name>wamv</name>
-          <link_name>base_link</link_name>
+          <link_name>wamv/base_link</link_name>
           <coeff_vector>.5 .5 .33</coeff_vector>
         </wind_obj>

File: vrx_gazebo/worlds/xacros/perception.xacro (robot description, xacro)
@@ -3,17 +3,22 @@
   <xacro:macro name="perception" params="**model_includes
                                          **object_sequence
-                                         ">
+                                         namespace:=wamv
+                                         competition:=vrx">
     <xacro:insert_block name="model_includes"/>"
       <plugin filename="libperception_scoring_plugin.so"
               name="perception_scoring_plugin">
       <!-- Parameters for ScoringPlugin base class -->
-      <vehicle>wamv</vehicle>
+      <vehicle>${namespace}</vehicle>
       <task_name>perception</task_name>
       <initial_state_duration>10.0</initial_state_duration>
       <ready_state_duration>10.0</ready_state_duration>
       <running_state_duration>300</running_state_duration>
+      <task_info_topic>/${competition}/task/info</task_info_topic>
+      <contact_debug_topic>/${competition}/debug/contact</contact_debug_topic>
+      <landmark_topic>/${competition}/perception/landmark</landmark_topic>
+      <per_plugin_exit_on_completion>true</per_plugin_exit_on_completion>
       <!-- Parameters for PopulationPlugin -->
       <loop_forever>false</loop_forever>
-      <frame>wamv</frame>
+      <frame>${namespace}</frame>
       <!-- Pose of each object is expressed relative to the body frame
            of the object named in the frame field - i.e., relative to

File: vrx_gazebo/worlds/xacros/stationkeeping.xacro (robot description, xacro)
@@ -1,11 +1,17 @@
 <?xml version="1.0"?>
 <world xmlns:xacro="http://ros.org/wiki/xacro">
-  <xacro:macro name="stationkeeping" params="**wp_markers lat:=21.31091 lon:=-157.88868 heading:=0.0">
+  <xacro:macro name="stationkeeping" params="**wp_markers lat:=21.31091 lon:=-157.88868 heading:=0.0 namespace:=wamv competition:=vrx">
     <plugin name="stationkeeping_scoring_plugin"
           filename="libstationkeeping_scoring_plugin.so">
-      <vehicle>wamv</vehicle>
+      <vehicle>${namespace}</vehicle>
       <task_name>stationkeeping</task_name>
+      <rms_error_topic>/${competition}/station_keeping/rms_error</rms_error_topic>
+      <pose_error_topic>/${competition}/station_keeping/pose_error</pose_error_topic>
+      <goal_topic>/${competition}/station_keeping/goal</goal_topic>
+      <task_info_topic>/${competition}/task/info</task_info_topic>
+      <contact_debug_topic>/${competition}/debug/contact</contact_debug_topic>
+      <per_plugin_exit_on_completion>true</per_plugin_exit_on_completion>
       <!-- Goal as Latitude, Longitude, Yaw -->
-      <goal_pose>${lat} ${lon} ${heading} </goal_pose>
+      <goal_pose>${lat} ${lon} ${heading}</goal_pose>
       <initial_state_duration>10</initial_state_duration>
       <ready_state_duration>10</ready_state_duration>
@@ -13,8 +19,8 @@
       <release_joints>
         <joint>
-          <name>wamv_external_pivot_joint</name>
+          <name>${namespace}_external_pivot_joint</name>
         </joint>
         <joint>
-          <name>wamv_external_riser</name>
+          <name>${namespace}_external_riser</name>
         </joint>
       </release_joints>

File: vrx_gazebo/worlds/xacros/wayfinding.xacro (robot description, xacro)
@@ -1,9 +1,18 @@
 <?xml version="1.0"?>
 <world xmlns:xacro="http://ros.org/wiki/xacro">
-  <xacro:macro name="wayfinding" params="**wp_markers **waypoints">
+  <xacro:macro name="wayfinding" params="**wp_markers
+                                         **waypoints
+                                         namespace:=wamv
+                                         competition:=vrx">
     <plugin name="wayfinding_scoring_plugin"
             filename="libwayfinding_scoring_plugin.so">
-      <vehicle>wamv</vehicle>
+      <vehicle>${namespace}</vehicle>
       <task_name>wayfinding</task_name>
+      <min_errors_topic>/${competition}/wayfinding/min_errors</min_errors_topic>
+      <mean_error_topic>/${competition}/wayfinding/mean_error</mean_error_topic>
+      <waypoints_topic>/${competition}/wayfinding/waypoints</waypoints_topic>
+      <task_info_topic>/${competition}/task/info</task_info_topic>
+      <contact_debug_topic>/${competition}/debug/contact</contact_debug_topic>
+      <per_plugin_exit_on_completion>true</per_plugin_exit_on_completion>
       <!-- Goal as Latitude, Longitude, Yaw -->
       <waypoints>
@@ -15,8 +24,8 @@
       <release_joints>
         <joint>
-          <name>wamv_external_pivot_joint</name>
+          <name>${namespace}_external_pivot_joint</name>
         </joint>
         <joint>
-          <name>wamv_external_riser</name>
+          <name>${namespace}_external_riser</name>
         </joint>
       </release_joints>

File: wamv_gazebo/urdf/dynamics/wamv_gazebo_dynamics_plugin.xacro (robot description, xacro)
@@ -1,9 +1,9 @@
 <?xml version="1.0"?>
 <robot xmlns:xacro="http://ros.org/wiki/xacro">
-  <xacro:macro name="usv_dynamics_gazebo" params="name">
+  <xacro:macro name="usv_dynamics_gazebo" params="name width:=2.4 length:=4.9">
     <!--Gazebo Plugin for simulating WAM-V dynamics-->
     <gazebo>
       <plugin name="usv_dynamics_${name}" filename="libusv_gazebo_dynamics_plugin.so">
-        <bodyName>base_link</bodyName>
+        <bodyName>${namespace}/base_link</bodyName>
         <!-- Must be same as the ocean model!-->
         <waterLevel>0</waterLevel>
@@ -26,6 +26,6 @@
         <!--<boatArea>2.2</boatArea>-->
         <hullRadius>0.213</hullRadius>
-        <boatWidth>2.4</boatWidth>
-        <boatLength>4.9</boatLength>
+        <boatWidth>${width}</boatWidth>
+        <boatLength>${length}</boatLength>
         <!-- Length discretization, AKA, "N" -->
         <length_n>2</length_n>

File: wamv_gazebo/urdf/sensors/wamv_3d_lidar.xacro (robot description, xacro)
@@ -10,4 +10,5 @@
     Y: Yaw orientation of the laser (from the laser's origin).
     post_Y: Yaw orientation of the post (from the post's origin).
+    post_z_from: Z position of the post's base.
     update_rate: frequency to publish output, hz
     vertical_lasers: number of vertical lasers which spin about Z to generate output
@@ -24,5 +25,5 @@
                                             x:=0.7 y:=0 z:=1.8
                                             R:=0 P:=0 Y:=0
-                                            post_Y:=0
+                                            post_Y:=0 post_z_from:=1.2965
                                             update_rate:=10 vertical_lasers:=16 samples:=1875 resolution:=0.1
                                             min_angle:=${-pi} max_angle:=${pi}
@@ -30,10 +31,10 @@
                                             max_range:=130 noise_stddev:=0.01">
     <!-- Define length variables for link positioning -->
-    <xacro:property name="platform_z" value="1.2965"/>
+    <xacro:property name="platform_z" value="${post_z_from}"/>
     <xacro:property name="post_to_post_arm_x" value="0.03"/>
     <xacro:property name="post_arm_to_lidar_x" value="0.04"/>
     <xacro:property name="post_arm_to_lidar_z" value="0.05"/>
     <!-- 3d lidar sensor -->
-    <link name="${name}_link">
+    <link name="${namespace}/${name}_link">
       <visual name="${name}_visual">
         <origin xyz="0 0 -0.035" rpy="0 0 0"/>
@@ -64,5 +65,5 @@
     <xacro:property name="post_radius" value="0.0076"/>
     <!-- Sensor post -->
-    <link name="${name}_post_link">
+    <link name="${namespace}/${name}_post_link">
       <visual>
         <geometry>
@@ -90,5 +91,5 @@
     </link>
     <!-- Sensor post arm -->
-    <link name="${name}_post_arm_link">
+    <link name="${namespace}/${name}_post_arm_link">
       <visual name="${name}_post_arm_visual">
         <origin xyz="-0.038 0 -0.003" rpy="${radians(-60)} 0 ${-pi/2}"/>
@@ -118,22 +119,22 @@
     <xacro:property name="post_z" value="${platform_z+post_length/2}"/>
     <xacro:property name="post_to_lidar_x" value="${post_to_post_arm_x+post_arm_to_lidar_x}"/>
-    <joint name="base_to_${name}_post_joint" type="fixed">
+    <joint name="${namespace}/base_to_${name}_post_joint" type="fixed">
       <origin xyz="${x-(post_to_lidar_x)*cos(post_Y)} ${y-(post_to_lidar_x)*sin(post_Y)} ${post_z}" rpy="0 0 ${post_Y}" />
-      <parent link="base_link" />
-      <child link="${name}_post_link" />
+      <parent link="${namespace}/base_link" />
+      <child link="${namespace}/${name}_post_link" />
     </joint>
     <!-- Sensor post to sensor post arm joint -->
-    <joint name="${name}_post_to_${name}_post_arm_joint" type="fixed">
+    <joint name="${namespace}/${name}_post_to_${name}_post_arm_joint" type="fixed">
       <origin xyz="${post_to_post_arm_x} 0 ${z-post_z-post_arm_to_lidar_z}" rpy="0 0 0" />
-      <parent link="${name}_post_link" />
-      <child link="${name}_post_arm_link" />
+      <parent link="${namespace}/${name}_post_link" />
+      <child link="${namespace}/${name}_post_arm_link" />
     </joint>
     <!-- Sensor post arm to lidar joint -->
-    <joint name="${name}_post_arm_to_${name}_joint" type="fixed">
+    <joint name="${namespace}/${name}_post_arm_to_${name}_joint" type="fixed">
       <origin xyz="${post_arm_to_lidar_x} 0 ${post_arm_to_lidar_z}" rpy="${R} ${P} ${Y-post_Y}" />
-      <parent link="${name}_post_arm_link" />
-      <child link="${name}_link" />
+      <parent link="${namespace}/${name}_post_arm_link" />
+      <child link="${namespace}/${name}_link" />
     </joint>
-    <gazebo reference="${name}_link">
+    <gazebo reference="${namespace}/${name}_link">
       <sensor type="gpu_ray" name="${name}_sensor">
         <update_rate>${update_rate}</update_rate>
@@ -171,5 +172,5 @@
     </gazebo>
     <!-- Set color of post -->
-    <gazebo reference="${name}_post_link">
+    <gazebo reference="${namespace}/${name}_post_link">
       <material>Gazebo/Black</material>
     </gazebo>

File: wamv_gazebo/urdf/sensors/wamv_camera.xacro (robot description, xacro)
@@ -1,12 +1,12 @@
 <?xml version="1.0"?>
 <robot xmlns:xacro="http://ros.org/wiki/xacro">
-  <xacro:macro name="wamv_camera" params="name x:=0.5 y:=0 z:=1.5 R:=0 P:=0 Y:=0 post_Y:=0">
+  <xacro:macro name="wamv_camera" params="name x:=0.5 y:=0 z:=1.5 post_z_from:=1.2965 R:=0 P:=0 Y:=0 post_Y:=0">
     <!-- Define length variables for link positioning -->
-    <xacro:property name="platform_z" value="1.2965"/>
+    <xacro:property name="platform_z" value="${post_z_from}"/>
     <xacro:property name="post_to_post_arm_x" value="0.03"/>
     <xacro:property name="post_arm_to_camera_x" value="0.02"/>
     <xacro:property name="post_arm_to_camera_z" value="0.027"/>
     <!-- Monocular Camera -->
-    <link name="${name}_link">
+    <link name="${namespace}/${name}_link">
       <visual name="${name}_visual">
         <origin xyz="-0.033 0 0" rpy="0 0 ${pi/2}"/>
@@ -41,5 +41,5 @@
     <!-- Define a link for the optical frame.  This will match the sensor frame and
          be oriented in the camera convention. -->
-    <link name="${name}_link_optical">
+    <link name="${namespace}/${name}_link_optical">
     </link>
     <!-- Define post length and mass based on desired z position of sensor -->
@@ -49,5 +49,5 @@
     <xacro:property name="post_radius" value="0.0076"/>
     <!-- Sensor post -->
-    <link name="${name}_post_link">
+    <link name="${namespace}/${name}_post_link">
       <visual>
         <geometry>
@@ -75,5 +75,5 @@
     </link>
     <!-- Sensor post arm -->
-    <link name="${name}_post_arm_link">
+    <link name="${namespace}/${name}_post_arm_link">
       <visual name="${name}_post_arm_visual">
         <origin xyz="-0.038 0 -0.003" rpy="${radians(-60)} 0 ${-pi/2}"/>
@@ -103,30 +103,30 @@
     <xacro:property name="post_z" value="${platform_z+post_length/2}"/>
     <xacro:property name="post_to_camera_x" value="${post_to_post_arm_x+post_arm_to_camera_x}"/>
-    <joint name="base_to_${name}_post_joint" type="fixed">
+    <joint name="${namespace}/base_to_${name}_post_joint" type="fixed">
       <origin xyz="${x-(post_to_camera_x)*cos(post_Y)} ${y-(post_to_camera_x)*sin(post_Y)} ${post_z}" rpy="0 0 ${post_Y}" />
-      <parent link="base_link" />
-      <child link="${name}_post_link" />
+      <parent link="${namespace}/base_link" />
+      <child link="${namespace}/${name}_post_link" />
     </joint>
     <!-- Sensor post to sensor post arm joint -->
-    <joint name="${name}_post_to_${name}_post_arm_joint" type="fixed">
+    <joint name="${namespace}/${name}_post_to_${name}_post_arm_joint" type="fixed">
       <origin xyz="${post_to_post_arm_x} 0 ${z-post_z-post_arm_to_camera_z}" rpy="0 0 0" />
-      <parent link="${name}_post_link" />
-      <child link="${name}_post_arm_link" />
+      <parent link="${namespace}/${name}_post_link" />
+      <child link="${namespace}/${name}_post_arm_link" />
     </joint>
     <!-- Sensor post arm to camera joint -->
-    <joint name="${name}_post_arm_to_${name}_joint" type="fixed">
+    <joint name="${namespace}/${name}_post_arm_to_${name}_joint" type="fixed">
       <origin xyz="${post_arm_to_camera_x} 0 ${post_arm_to_camera_z}" rpy="${R} ${P} ${Y-post_Y}" />
-      <parent link="${name}_post_arm_link" />
-      <child link="${name}_link" />
+      <parent link="${namespace}/${name}_post_arm_link" />
+      <child link="${namespace}/${name}_link" />
     </joint>
     <!-- Camera to optical frame joint.  This is oriented to convert between ENU
          and camera conventions -->
-    <joint name="${name}_to_${name}_link_optical_joint" type="fixed">
+    <joint name="${namespace}/${name}_to_${name}_link_optical_joint" type="fixed">
       <origin xyz="0 0 0" rpy="${-pi/2} 0 ${-pi/2}" />
-      <parent link="${name}_link" />
-      <child link="${name}_link_optical" />
+      <parent link="${namespace}/${name}_link" />
+      <child link="${namespace}/${name}_link_optical" />
     </joint>
     <!-- Gazebo camera setup -->
-    <gazebo reference="${name}_link">
+    <gazebo reference="${namespace}/${name}_link">
       <sensor type="camera" name="${name}_sensor">
         <update_rate>30.0</update_rate>
@@ -168,5 +168,5 @@
     </gazebo>
     <!-- Set color of post -->
-    <gazebo reference="${name}_post_link">
+    <gazebo reference="${namespace}/${name}_post_link">
       <material>Gazebo/Black</material>
     </gazebo>

File: wamv_gazebo/urdf/sensors/wamv_gps.xacro (robot description, xacro)
@@ -1,6 +1,6 @@
 <?xml version="1.0" encoding="UTF-8"?>
 <robot xmlns:xacro="http://ros.org/wiki/xacro">
-  <xacro:macro name="wamv_gps" params="name:=gps x:=0.3 y:=0 z:=1.3 R:=0 P:=0 Y:=0">
-    <link name="${name}_link">
+  <xacro:macro name="wamv_gps" params="name:=gps x:=0.3 y:=0 z:=1.3 R:=0 P:=0 Y:=0 lat:=-33.724223 lon:=150.679736 elev:=0.0 update_rate:=15">
+    <link name="${namespace}/${name}_link">
       <visual name="${name}_visual">
         <geometry>
@@ -25,16 +25,16 @@
       </inertial>
     </link>
-    <joint name="${name}_joint" type="revolute">
+    <joint name="${namespace}/${name}_joint" type="revolute">
       <axis xyz="0 0 1"/>
       <limit effort="1000.0" lower="0.0" upper="0" velocity="0"/>
       <origin xyz="${x} ${y} ${z}" rpy="${R} ${P} ${Y}" />
-      <parent link="base_link" />
-      <child link="${name}_link" />
+      <parent link="${namespace}/base_link" />
+      <child link="${namespace}/${name}_link" />
     </joint>
     <gazebo>
       <plugin name="gps_plugin_${name}" filename="libhector_gazebo_ros_gps.so">
-        <updateRate>15.0</updateRate>
+        <updateRate>${update_rate}</updateRate>
         <alwaysOn>true</alwaysOn>
-        <bodyName>${name}_link</bodyName>
+        <bodyName>${namespace}/${name}_link</bodyName>
         <!-- Manually prepend namespace to tf frame. -->
         <frameId>${namespace}/${name}_link</frameId>
@@ -47,8 +47,8 @@
         <velocityTopicName>${namespace}/${sensor_namespace}gps/gps/fix_velocity</velocityTopicName>
         <!-- Location of origin of Gazebo Sand Island map -->
-        <referenceLatitude>21.30996</referenceLatitude>
-        <referenceLongitude>-157.8901</referenceLongitude>
-        <referenceAltitude>0</referenceAltitude>
-        <referenceHeading>90</referenceHeading>
+        <referenceLatitude>${lat}</referenceLatitude>
+        <referenceLongitude>${lon}</referenceLongitude>
+        <referenceAltitude>${elev}</referenceAltitude>
+        <referenceHeading>270</referenceHeading>
         <offset>0.0 0.0 0.0</offset>
         <drift>0.0 0.0 0.0</drift>

File: wamv_gazebo/urdf/sensors/wamv_imu.xacro (robot description, xacro)
@@ -1,6 +1,6 @@
 <?xml version="1.0"?>
 <robot xmlns:xacro="http://ros.org/wiki/xacro">
-  <xacro:macro name="wamv_imu" params="name:=imu x:=0.3 y:=0.5 z:=1.3 R:=0 P:=0 Y:=0">
-    <link name="${name}_link">
+  <xacro:macro name="wamv_imu" params="name:=imu x:=0.3 y:=0.5 z:=1.3 R:=0 P:=0 Y:=0 update_rate:=15">
+    <link name="${namespace}/${name}_link">
       <visual name="${name}_visual">>
         <geometry>
@@ -16,15 +16,15 @@
       </inertial>
     </link>
-    <joint name="${name}_joint" type="revolute">
+    <joint name="${namespace}/${name}_joint" type="revolute">
       <axis xyz="0 0 1"/>
       <limit effort="1000.0" lower="0.0" upper="0" velocity="0"/>
       <origin xyz="${x} ${y} ${z}" rpy="${R} ${P} ${Y}"/>
-      <parent link="base_link"/>
-      <child link="${name}_link"/>
+      <parent link="${namespace}/base_link"/>
+      <child link="${namespace}/${name}_link"/>
     </joint>
     <gazebo>
       <plugin name="imu_plugin_${name}" filename="libhector_gazebo_ros_imu.so">
-        <updateRate>15.0</updateRate>
-        <bodyName>${name}_link</bodyName>
+        <updateRate>${update_rate}</updateRate>
+        <bodyName>${namespace}/${name}_link</bodyName>
         <topicName>${namespace}/${sensor_namespace}imu/imu/data</topicName>
         <serviceName>${namespace}/${sensor_namespace}imu_service</serviceName>

File: wamv_gazebo/urdf/sensors/wamv_pinger.xacro (robot description, xacro)
@@ -1,6 +1,6 @@
 <?xml version="1.0"?>
 <robot xmlns:xacro="http://ros.org/wiki/xacro">
-  <xacro:macro name="wamv_pinger" params="name:='pinger' position:='0 0 0' orientation:='0 0 0'">
-    <link name="${name}">
+  <xacro:macro name="wamv_pinger" params="name:='pinger' frameId:='wamv/pinger' position:='0 0 0' orientation:='0 0 0'">
+    <link name="${namespace}/${name}">
       <visual>
         <origin xyz="0 0 0" rpy="0 0 0" />
@@ -16,12 +16,12 @@
       </collision>
     </link>
-    <joint name="${name}_pinger_joint" type="fixed">
+    <joint name="${namespace}/${name}_pinger_joint" type="fixed">
       <origin xyz="${position}" rpy="${orientation}"/>
-      <parent link="base_link"/>
-      <child link="${name}"/>
+      <parent link="${namespace}/base_link"/>
+      <child link="${namespace}/${name}"/>
     </joint>
     <gazebo>
       <plugin name="pinger_plugin" filename="libusv_gazebo_acoustic_pinger_plugin.so">
-        <frameId>wamv/pinger</frameId>
+        <frameId>${frameId}</frameId>
         <topicName>${namespace}/${sensor_namespace}${pinger_namespace}${name}/range_bearing</topicName>
         <setPositionTopicName>${namespace}/${sensor_namespace}${pinger_namespace}${name}/set_pinger_position</setPositionTopicName>

File: wamv_gazebo/urdf/thruster_layouts/wamv_gazebo_thruster_config.xacro (robot description, xacro)
@@ -1,13 +1,13 @@
 <?xml version="1.0"?>
 <plugin xmlns:xacro="http://ros.org/wiki/xacro">
-  <xacro:macro  name="wamv_gazebo_thruster_config" params="name">
+  <xacro:macro  name="wamv_gazebo_thruster_config" params="name enable_angle:=true">
     <thruster>
       <!-- Required Parameters -->
-      <linkName>${name}_propeller_link</linkName>
-      <propJointName>${name}_engine_propeller_joint</propJointName>
-      <engineJointName>${name}_chasis_engine_joint</engineJointName>
+      <linkName>${namespace}/${name}_propeller_link</linkName>
+      <propJointName>${namespace}/${name}_engine_propeller_joint</propJointName>
+      <engineJointName>${namespace}/${name}_chasis_engine_joint</engineJointName>
       <cmdTopic>${thruster_namespace}${name}_thrust_cmd</cmdTopic>
       <angleTopic>${thruster_namespace}${name}_thrust_angle</angleTopic>
-      <enableAngle>true</enableAngle>
+      <enableAngle>${enable_angle}</enableAngle>
       <!-- Optional Parameters -->
       <mappingType>1</mappingType>
