Commit message: updated vrx code

File: wamv_gazebo/urdf/wamv_gazebo.urdf.xacro (robot description, xacro)
@@ -12,8 +12,10 @@
   <xacro:arg name="vrx_sensors_enabled" default="false" />
   <xacro:arg name="pinger_enabled" default="false" />
+  <xacro:arg name="ball_shooter_enabled" default="false" />
   <xacro:arg name="thruster_namespace" default="thrusters/"/>
   <xacro:arg name="camera_namespace" default="cameras/"/>
   <xacro:arg name="sensor_namespace" default="sensors/"/>
   <xacro:arg name="pinger_namespace" default="pingers/"/>
+  <xacro:arg name="shooter_namespace" default="shooters/"/>
   <!-- Note: this is only used for some sensors that do not correctly use the
   robotNamespace parameter -->
@@ -23,4 +25,5 @@
   <xacro:property name="sensor_namespace" value="$(arg sensor_namespace)" scope="global" />
   <xacro:property name="pinger_namespace" value="$(arg pinger_namespace)" scope="global" />
+  <xacro:property name="shooter_namespace" value="$(arg shooter_namespace)" scope="global" />
   <xacro:property name="namespace" value="$(arg namespace)" scope="global" />
   <!-- Sensor yaml file -->
@@ -62,5 +65,5 @@
       <link name="wamv_external_link"/>
       <joint name="wamv_external_pivot_joint" type="universal">
-        <parent>wamv::base_link</parent>
+        <parent>wamv::wamv/base_link</parent>
         <child>wamv_external_link</child>
         <axis>
@@ -119,4 +122,8 @@
       <xacro:wamv_pinger name="pinger" position="1.0 0 -1.0" />
     </xacro:if>
+    <!-- Add ball shooter (default pitch angle: -15 deg) -->
+    <xacro:if value="$(arg ball_shooter_enabled)">
+      <xacro:wamv_ball_shooter name="ball_shooter" position="0.54 0.30 1.296" orientation="0 -0.261799 0"/>
+    </xacro:if>
     <!-- ==== VRX sensor configuration ==== -->
     <xacro:if value="$(arg vrx_sensors_enabled)">
@@ -137,4 +144,6 @@
       <!-- Add pinger -->
       <xacro:wamv_pinger name="pinger" position="1.0 0 -1.0" />
+      <!-- Add ball shooter (default pitch angle: -15 deg) -->
+      <xacro:wamv_ball_shooter name="ball_shooter" position="0.54 0.30 1.296" orientation="0 -0.261799 0"/>
     </xacro:if>
   </xacro:unless>

Commit message: modified example_course to release locked joints

File: vrx_gazebo/worlds/example_course.world.xacro (robot description, xacro)
@@ -56,4 +56,21 @@
       <pose>-420 295 0 0 0 -2.04</pose>
     </include>
+    <plugin filename="libscoring_plugin.so"
+            name="scoring_plugin">
+      <!-- Parameters for ScoringPlugin base class -->
+      <vehicle>wamv</vehicle>
+      <task_name>none</task_name>
+      <initial_state_duration>3.0</initial_state_duration>
+      <ready_state_duration>0.0</ready_state_duration>
+      <running_state_duration>3000</running_state_duration>
+      <release_joints>
+        <joint>
+          <name>wamv_external_pivot_joint</name>
+        </joint>
+        <joint>
+          <name>wamv_external_riser</name>
+        </joint>
+      </release_joints>
+    </plugin>
   </world>
 </sdf>
