Commit message: added mil lidar and engine

File: wamv_gazebo/urdf/components/mil_3d_lidar.xacro (robot description, xacro)
@@ -36,5 +36,5 @@
     <xacro:property name="post_arm_to_lidar_z" value="0.05"/>
     <!-- 3d lidar sensor -->
-    <link name="${name}_link">
+    <link name="${name}">
       <visual name="${name}_visual">
         <origin xyz="0 0 -0.035" rpy="0 0 0"/>
@@ -134,7 +134,7 @@
       <origin xyz="${post_arm_to_lidar_x} 0 ${post_arm_to_lidar_z}" rpy="${R} ${P} ${Y-post_Y}" />
       <parent link="${name}_post_arm_link" />
-      <child link="${name}_link" />
+      <child link="${name}" />
     </joint>
-    <gazebo reference="${name}_link">
+    <gazebo reference="${name}">
       <sensor type="gpu_ray" name="${name}_sensor">
         <update_rate>${update_rate}</update_rate>
@@ -166,6 +166,6 @@
         <plugin name="${name}_plugin" filename="libgazebo_ros_velodyne_gpu_laser.so">
           <topicName>velodyne_points</topicName>
-          <frameName>${name}_link</frameName>
-          <min_intensity>0</min_intensity>velodyne
+	  <frameName>${name}</frameName>
+          <min_intensity>0</min_intensity>
         </plugin>
       </sensor>
