Commit message: added transmission to engine.xacro

File: wamv_description/urdf/thrusters/engine.xacro (robot description, xacro)
@@ -55,7 +55,18 @@
       <child link="${namespace}/${prefix}_propeller_link"/>
       <origin rpy="0 0 0" xyz="-0.278156 0 -0.509371"/>
-      <limit effort="100" velocity="100" />
+      <limit effort="400" velocity="100" />
       <dynamics friction="0.05" damping="0.05" />
     </joint>
+    <transmission name="${namespace}/${prefix}_thruster_transmission">
+      <type>transmission_interface/SimpleTransmission</type>
+      <actuator name="${namespace}/${prefix}_motor">
+        <!-- Linear Mapping from force to actuator "effort" (motor command) such that
+             -->
+        <mechanicalReduction>1.35</mechanicalReduction>
+      </actuator>
+      <joint name="${namespace}/${prefix}_engine_propeller_joint">
+        <hardwareInterface>hardware_interface/EffortJointInterface</hardwareInterface>
+      </joint>
+    </transmission>
   </xacro:macro>
 </robot>

Commit message: Corrected engine.xacro

File: wamv_description/urdf/thrusters/engine.xacro (robot description, xacro)
@@ -58,15 +58,4 @@
       <dynamics friction="0.05" damping="0.05" />
     </joint>
-    <transmission name="${namespace}/${prefix}_thruster_transmission">
-      <type>transmission_interface/SimpleTransmission</type>
-      <actuator name="${namespace}/${prefix}_motor">
-        <!-- Linear Mapping from force to actuator "effort" (motor command) such that
-             -->
-        <mechanicalReduction>1.35</mechanicalReduction>
-      </actuator>
-      <joint name="${namespace}/${prefix}_engine_propeller_joint">
-        <hardwareInterface>hardware_interface/EffortJointInterface</hardwareInterface>
-      </joint>
-    </transmission>
   </xacro:macro>
 </robot>
