Commit message: mil_mech_reduct

File: wamv_description/urdf/thrusters/mil_engine.xacro (robot description, xacro)
@@ -2,5 +2,5 @@
 <robot xmlns:xacro="http://ros.org/wiki/xacro" name="wam-v-two-engines">
   <!-- Macro for inserting an engine with its propeller. -->
-  <xacro:macro name="mil_engine" params="prefix position:='0 0 0' orientation:='0 0 0'">
+  <xacro:macro name="mil_engine" params="prefix position:='0 0 0' orientation:='0 0 0' mech_reduction:='1.35'">
     <link name="${prefix}_engine_link">
       <visual>
@@ -63,5 +63,5 @@
         <!-- Linear Mapping from force to actuator "effort" (motor command) such that
              -->
-        <mechanicalReduction>1.35</mechanicalReduction>
+	<mechanicalReduction>${mech_reduction}</mechanicalReduction>
       </actuator>
       <joint name="${prefix}_engine_propeller_joint">
